File: EAGLE/datapath/schematics/datapath.sch (EAGLE design)
At the start: 10 parts, among them IC1 74LS08N, IC2 7432N, IC3 74LS08N, IC4 74LS08N, IC5 7432N

Commit message: completed datapath
Parts:
- added HR: 74LS93N, 74xx-us:74LS93N
- added HR_ADDER: 74LS283N, 74xx-us:74LS283N
- added IC6: 7432N, 74xx-us:7432N
- added IC7: 7400N, 74xx-us:7400N
- added MRDN: 74LS109N, 74xx-us:74LS109N
Connections:
- new net 5V: HR_ADDERA.C0, MRDNA.J
- new net ADD_HR_LG: IC6B.I0
- new net AMPM: MRDNA.Q
- new net CLR: IC7A.O, MRDNA.CLR
- new net HR0: HR_ADDERA.S1
- new net HR1: HR_ADDERA.S2
- new net HR2: HR_ADDERA.S3
- new net HR3: HR_ADDERA.S4
- new net HR_INT_0: HRA.CKB, HRA.QA, HR_ADDERA.A1
- new net HR_INT_1: HRA.QB, HR_ADDERA.A2
- new net HR_INT_2: HRA.QC, HR_ADDERA.A3, IC4D.I0
- new net HR_INT_3: HRA.QD, HR_ADDERA.A4, IC4D.I1
- new net HR_OVF: IC4D.O, IC6A.I1, IC6B.I1
- new net HR_RST: HRA.R0(1), HRA.R0(2), IC6A.O
- new net N$1: MRDNA.PRE
- new net T_MRDN: IC6B.O, MRDNA.CLK
- net GND: now also HR_ADDERA.B1, HR_ADDERA.B2, HR_ADDERA.B3, HR_ADDERA.B4, MRDNA.K
- net HR_INC: now also HRA.CKA
- net RST: now also IC6A.I0, IC7A.I0, IC7A.I1
